File: KiCad-7 Files/power.kicad_sch (KiCad schematic)
At the start: 5 parts, among them Q1 PJA3407_R1_00001

Commit message: Add files via upload
upload new kicad 7 files with certification mark
Parts:
- D1: value 3V3 -> CZRU52C3V3
- D2: value BLU led -> APTD2012LQBC/D
Other:
- note added: "3V3"
- note added: "BLU LED"
- note removed: "CZRU52C3V3"
Changed lines of the file:
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@@
     (stroke (width 0) (type default))
   )
-  (text "CZRU52C3V3" (at 150.876 93.98 0)
+  (text "3V3" (at 152.654 92.456 0)
+    (effects (font (size 1 1)) (justify left bottom))
+  )
+  (text "BLU LED\n" (at 166.37 105.41 0)
     (effects (font (size 1 1)) (justify left bottom))
   )
@@
       (effects (font (size 1.27 1.27)) (justify right))
     )
-    (property "Value" "BLU led" (at 166.37 103.1874 90)
+    (property "Value" "APTD2012LQBC/D" (at 166.37 103.1874 90)
       (effects (font (size 1.27 1.27)) (justify right))
     )
@@
       (effects (font (size 1.27 1.27)) (justify left))
     )
-    (property "Value" "3V3" (at 152.4 90.932 90)
-      (effects (font (size 1.27 1.27)) (justify left))
+    (property "Value" "CZRU52C3V3" (at 152.654 90.424 90)
+      (effects (font (size 0.762 0.762)) (justify left))
     )
     (property "Footprint" "Diode_SMD:D_0603_1608Metric" (at 149.86 90.17 0)
